Commit message: CCTA 2013

File: CCTA 2023/Exo/description.urdf (robot description, URDF)
Before this commit: robot EXO_TAO, 4 links, 3 joints
Links:
- link lr_leg: mass None -> 1
- link lr_shank: mass None -> 1
Joints:
- joint jr_knee: origin xyz=0.0 0.0 0.0 rpy=0.0 0.0 0.0 -> xyz=0.265 0.0 0.42 rpy=0.0 0.0 0.0
- joint r_bar: limit (none) -> lower=-0.785 upper=0.785 effort=3.0 velocity=4.0; origin xyz=0.0 0.0 0.84 rpy=0.0 0.0 0.0 -> xyz=0.0 0.0 0.84 rpy=3.14 0.0 0.0
- joint r_knee: limit (none) -> lower=0.0 upper=1.57 effort=3.0 velocity=4.0; origin xyz=0.0 0.0 0.0 rpy=3.14 0.0 0.0 -> xyz=-0.03 0.0 0 rpy=0 0.0 0.0
