Commit message: CCTA 2023

File: CCTA 2023/Exo/description_v1.urdf (robot description, URDF)
Before this commit: robot EXO_TAO, 9 links, 8 joints
Joints:
- joint l_hip: origin xyz=0.0 0.0 0.84 rpy=3.14 0.0 0.0 -> xyz=0.0 0.0 0.84 rpy=3.1415 0.0 0.0
- joint l_knee: limit lower=0.0 upper=1.57 effort=3.0 velocity=4.0 -> lower=0.0 upper=1.5707 effort=3.0 velocity=4.0
- joint r_hip: origin xyz=0.0 0.0 0.84 rpy=3.14 0.0 0.0 -> xyz=0.0 0.0 0.84 rpy=3.1415 0.0 0.0
- joint r_knee: limit lower=0.0 upper=1.57 effort=3.0 velocity=4.0 -> lower=0.0 upper=1.5707 effort=3.0 velocity=4.0

Commit message: CCTA 2023

File: CCTA 2023/Exo/description_v1.urdf (robot description, URDF)
Before this commit: robot EXO_TAO, 9 links, 8 joints
Links:
- link ll_hip: mass None -> 1
- link ll_knee: mass None -> 1
- link lr_hip: mass None -> 1
- link lr_knee: mass None -> 1
